File: Knave+Death.sch (KiCad schematic (older format))
At the start: 42 parts, among them J1 OUT0_3.5mm, J2 OUT1_3.5mm, J3 OUT2_3.5mm, J4 PWR_IN_PHNX, J5 OUT3_3.5mm, J6 E0_3.5mm, J7 E1_3.5mm, SW1 SW_SPDT, U1 LM324, U2 LM358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

Commit message: laid out some hypothetical components:
Parts:
- RV1: footprint HammerheadAudio:R_THT_P7.62 -> Potentiometer_THT:Potentiometer_Piher_PT-6-V_Vertical
- U2: footprint Package_DIP:DIP-14_W7.62mm_Socket -> Package_DIP:DIP-8_W7.62mm_Socket
Changed lines of the file:
@@
 EESchema Schematic File Version 4
-LIBS:CV_To_PWM_Converter-cache
+LIBS:Knave+Death-cache
 EELAYER 29 0
 EELAYER END
@@
 F 0 "RV1" H 5730 5804 50  0000 R CNN
 F 1 "1M" H 5730 5895 50  0000 R CNN
-F 2 "HammerheadAudio:R_THT_P7.62" H 5800 5850 50  0001 C CNN
+F 2 "Potentiometer_THT:Potentiometer_Piher_PT-6-V_Vertical" H 5800 5850 50  0001 C CNN
 F 3 "~" H 5800 5850 50  0001 C CNN
 	1    5800 5850
@@
 F 0 "U2" H 1150 4817 50  0000 C CNN
 F 1 "LM358" H 1150 4726 50  0000 C CNN
-F 2 "Package_DIP:DIP-14_W7.62mm_Socket" H 1100 4550 50  0001 C CNN
+F 2 "Package_DIP:DIP-8_W7.62mm_Socket" H 1100 4550 50  0001 C CNN
 F 3 "http://www.ti.com/lit/ds/symlink/lm2902-n.pdf" H 1200 4650 50  0001 C CNN
 	1    1150 4450
@@
 F 0 "U2" H 1150 5667 50  0000 C CNN
 F 1 "LM358" H 1150 5576 50  0000 C CNN
-F 2 "Package_DIP:DIP-14_W7.62mm_Socket" H 1100 5400 50  0001 C CNN
+F 2 "Package_DIP:DIP-8_W7.62mm_Socket" H 1100 5400 50  0001 C CNN
 F 3 "http://www.ti.com/lit/ds/symlink/lm2902-n.pdf" H 1200 5500 50  0001 C CNN
 	2    1150 5300
@@
 F 0 "U2" H 7908 1696 50  0000 L CNN
 F 1 "LM358" H 7908 1605 50  0000 L CNN
-F 2 "Package_DIP:DIP-14_W7.62mm_Socket" H 7900 1750 50  0001 C CNN
+F 2 "Package_DIP:DIP-8_W7.62mm_Socket" H 7900 1750 50  0001 C CNN
 F 3 "http://www.ti.com/lit/ds/symlink/lm2902-n.pdf" H 8000 1850 50  0001 C CNN
 	3    7950 1650
